File: pcb/PETKey_Arduino.brd (EAGLE design)
At the start: 35.6 x 53.3 mm, 6 parts, among them X2 KB_PORT_PET

Commit message: Fix incorrect XPT mappings
Parts:
- IC1: value (none) -> MT8812
Connections:
- removed net CLK: SV1.21
- removed net NOTUSED0: IC1.33
- removed net NOTUSED1: IC1.28
- removed net OE: SV1.22
Changed lines of the file:
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@@
 <attribute name="OC_NEWARK" value="unknown" x="10.16" y="24.13" size="1.778" layer="27" rot="R90" display="off"/>
 </element>
-<element name="IC1" library="MT8812" package="DIP40" value="" x="21.59" y="25.4" rot="R270"/>
+<element name="IC1" library="MT8812" package="DIP40" value="MT8812" x="21.59" y="25.4" rot="R270"/>
 <element name="X2" library="commodore" package="MA20-1_KEYED" value="KB_PORT_PET" x="33.02" y="24.13" rot="R90"/>
 </elements>
@@
 <contactref element="X2" pad="1"/>
 </signal>
-<signal name="CLK">
-<contactref element="SV1" pad="21"/>
-</signal>
-<signal name="OE">
-<contactref element="SV1" pad="22"/>
-</signal>
 <signal name="VCC">
 <contactref element="C1" pad="1"/>
@@
 <wire x1="31.75" y1="6.35" x2="33.02" y2="5.08" width="0.254" layer="16"/>
 </signal>
-<signal name="NOTUSED0">
-<contactref element="IC1" pad="33"/>
-</signal>
-<signal name="NOTUSED1">
-<contactref element="IC1" pad="28"/>
-</signal>
 </signals>
